File: Projects/Mouse Dongle Card/Electrical Schematic/Mouse Dongle Card.kicad_pcb (KiCad board)
At the start: 2 copper layers, 26 x 27.9 mm, 10 parts, among them J1 692121330100, P1 USB_C_Plug

Commit message: Fixed for manufacturing
Routing:
- net GND: track 29.5 -> 33.7 mm, vias 8 -> 10
- net VBUS: track 6.38 -> 6.48 mm, vias 0 -> 2
Changed lines of the file:
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@@
 		(tenting front back)
 		(pcbplotparams
-			(layerselection 0x00000000_00000000_55555555_57555550)
+			(layerselection 0x00000000_00000000_55555555_5f5555ff)
 			(plot_on_all_layers_selection 0x00000000_00000000_00000000_00000000)
 			(disableapertmacros no)
@@
 			(crossoutdnponfab yes)
 			(subtractmaskfromsilk no)
-			(outputformat 3)
+			(outputformat 1)
 			(mirror no)
 			(drillshape 0)
 			(scaleselection 1)
-			(outputdirectory "")
+			(outputdirectory "../Gerbers/")
 		)
 	)
@@
 		(tags "capacitor handsolder")
 		(property "Reference" "C1"
-			(at 0 -1.85 90)
+			(at -1.58 -2.4 180)
 			(layer "F.SilkS")
 			(effects
@@
 	)
 	(segment
+		(start 100.65 133.2)
+		(end 100.65 135.29)
+		(width 0.6)
+		(layer "F.Cu")
+		(net 1)
+	)
+	(segment
 		(start 102.59 121.95)
 		(end 102.6 121.96)
 		(width 1)
+		(layer "F.Cu")
+		(net 1)
+	)
+	(segment
+		(start 115.95 133.21)
+		(end 115.95 135.3)
+		(width 0.6)
 		(layer "F.Cu")
 		(net 1)
@@
 	)
 	(via
+		(at 115.95 133.21)
+		(size 0.6)
+		(drill 0.3)
+		(layers "F.Cu" "B.Cu")
+		(free yes)
+		(net 1)
+	)
+	(via
+		(at 100.65 133.2)
+		(size 0.6)
+		(drill 0.3)
+		(layers "F.Cu" "B.Cu")
+		(free yes)
+		(net 1)
+	)
+	(via
 		(at 113.5245 121.5315)
 		(size 0.5)
@@
 	)
 	(segment
-		(start 106.642 124.2)
+		(start 107.05 123.95)
+		(end 106.8 124.2)
+		(width 0.4)
+		(layer "F.Cu")
+		(net 3)
+	)
+	(segment
+		(start 106.8 124.2)
 		(end 106.4 124.2)
 		(width 0.4)
@@
 	)
 	(segment
-		(start 107.05 123.792)
-		(end 106.642 124.2)
+		(start 107.05 123.95)
+		(end 107.05 123)
 		(width 0.4)
 		(layer "F.Cu")
 		(net 3)
 	)
-	(segment
-		(start 107.05 123)
-		(end 107.05 123.792)
-		(width 0.4)
-		(layer "F.Cu")
+	(via
+		(at 109.25 124.25)
+		(size 0.5)
+		(drill 0.3)
+		(layers "F.Cu" "B.Cu")
+		(net 3)
+	)
+	(via
+		(at 107.05 123.95)
+		(size 0.5)
+		(drill 0.3)
+		(layers "F.Cu" "B.Cu")
 		(net 3)
 	)
@@
 	)
 	(segment
+		(start 109.25 124.25)
+		(end 109.1 124.4)
+		(width 0.2)
+		(layer "B.Cu")
+		(net 3)
+	)
+	(segment
 		(start 109.1 124.4)
 		(end 107.5 124.4)
@@
 	(segment
 		(start 109.55 123.95)
-		(end 109.1 124.4)
+		(end 109.25 124.25)
 		(width 0.2)
 		(layer "B.Cu")
@@
 	)
 	(segment
+		(start 106.7 125.05)
+		(end 107.55 124.2)
+		(width 0.2)
+		(layer "F.Cu")
+		(net 15)
+	)
+	(segment
+		(start 102.6 125.05)
+		(end 100.1 125.05)
+		(width 0.2)
+		(layer "F.Cu")
+		(net 15)
+	)
+	(segment
+		(start 100.1 125.45)
+		(end 100.1 125.05)
+		(width 0.2)
+		(layer "F.Cu")
+		(net 15)
+	)
+	(segment
+		(start 106.1 125.05)
+		(end 106.7 125.05)
+		(width 0.2)
+		(layer "F.Cu")
+		(net 15)
+	)
+	(segment
 		(start 107.55 124.2)
 		(end 107.55 123)
@@
 		(net 15)
 	)
-	(segment
-		(start 107.071446 124.678554)
-		(end 107.55 124.2)
-		(width 0.2)
-		(layer "F.Cu")
-		(net 15)
-	)
-	(segment
-		(start 100.1 125.45)
-		(end 100.1 125.05)
-		(width 0.2)
-		(layer "F.Cu")
-		(net 15)
-	)
-	(segment
-		(start 101.38 125.05)
-		(end 100.1 125.05)
-		(width 0.2)
-		(layer "F.Cu")
-		(net 15)
-	)
 	(via
-		(at 101.38 125.05)
+		(at 102.6 125.05)
 		(size 0.6)
 		(drill 0.3)
@@
 	)
 	(via
-		(at 107.071446 124.678554)
+		(at 106.1 125.05)
 		(size 0.6)
 		(drill 0.3)
@@
 	)
 	(segment
-		(start 106.7 125.05)
-		(end 107.071446 124.678554)
+		(start 106.1 125.05)
+		(end 102.6 125.05)
 		(width 0.2)
 		(layer "B.Cu")
-		(net 15)
-	)
-	(segment
-		(start 101.38 125.05)
-		(end 106.7 125.05)
-		(width 0.2)
-		(layer "B.Cu")
-		(net 15)
-	)
-	(segment
-		(start 101.39 125.04)
-		(end 101.38 125.05)
-		(width 0.2)
-		(layer "B.Cu")
